File: Hardware/USB Mux-v0.2.brd (EAGLE design)
At the start: 13.1 x 37.1 mm, 13 parts, among them U1 NCN9252, U2 XC6206P332MR

Commit message: PCB update, optional or'ing circuit
Routing:
- net N$11: track 14.6 -> 17.3 mm, vias 2 -> 3
- net GND: track 11.5 -> 13.9 mm, vias 30 -> 46
- net N$13: track 3.60 -> 6.04 mm, vias 0 -> 1
- net SEL0: track 3.25 -> 1.11 mm
- net N$12: track 9.36 -> 10.6 mm, vias 0 -> 1
- net SEL1: track 1.99 -> 1.07 mm
- net VCC: track 33.7 -> 33.8 mm, vias 1 -> 2
Other:
- board text added: "+3.3V"
- board text added: "D+"
- board text added: "D-"
- board text added: "GND"
- board text added: "S0"
- board text added: "S1"
- board text added: "VUSB"
